File: MATRIX-1.4-IV-T13-450W4L-COMPLEX-2/MATRIX-1.4-IV-T13-450W4L.kicad_sch (KiCad schematic)
At the start: 185 parts, among them Q201 2N5401, Q202 2N5551, Q203 2N5551, Q301 2N5551, Q401 2N5551, Q402 2N5551, Q403 MJE340, Q404 MJE350, Q405 MJE350, Q406 MJE340, Q407 MJE15032, Q408 MJE15033, Q409 2SC5200, Q410 2SA1943, Q4111 MJL21194, Q4112 MJL21194, Q4113 MJL21194, Q4114 MJL21194, Q4115 MJL21194, Q4121 MJL21193, Q4122 MJL21193, Q4123 MJL21193, Q4124 MJL21193, Q4125 MJL21193, Q501 2N5401, Q502 2N5551, Q503 2N5401, Q504 2N5551, Q505 2N5551, Q506 2N5401, Q507 2N5551, Q508 2N5551, Q509 TIP41C

Commit message: Routine Update Thu Jun  2 11:27:20 AM WIB 2022
Parts:
- C301, C401, C503: footprint MATRIX_1.4:CAPACITOR_AE_D5.08mm -> MATRIX_1.4:CAPACITOR_AE_D7.62mm
- D411, D412: footprint MATRIX_1.4:D_5KP_P12.70mm_Horizontal -> MATRIX_1.4:DIODE_AXIAL_SMALL_GE
- Q405: footprint MATRIX_1.4:TO-225-MIRRORED -> MATRIX_1.4:TO-225
- R514: footprint MATRIX_1.4:RESISTOR_AXIAL_0.5W -> MATRIX_1.4:RESISTOR_AXIAL_0.25W
- S1: renamed from S501; footprint MATRIX_1.4:Relay_SPDT_RAYEX-L90 -> Relay_THT:Relay_SPST_RAYEX-L90A
- renumbered R303 to R304, R304 to R305, R305 to R306, R306 to R307, R307 to R308, R4141 to R40141, R4142 to R40142, R4143 to R40143, R4144 to R40144, R4151 to R40151, R4152 to R40152, R4161 to R40161, R417 to R4017, R418 to R4018, R4205 to R4206
Changed lines of the file:
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@@
     (property "Reference" "D412" (id 0) (at 349.25 144.78 90))
     (property "Value" "10A03" (id 1) (at 349.25 147.32 90))
-    (property "Footprint" "MATRIX_1.4:D_5KP_P12.70mm_Horizontal" (id 2) (at 342.9 146.05 0)
+    (property "Footprint" "MATRIX_1.4:DIODE_AXIAL_SMALL_GE" (id 2) (at 342.9 146.05 0)
       (effects (font (size 1.27 1.27)) hide)
     )
@@
     (property "Reference" "C401" (id 0) (at 165.1 73.66 0))
     (property "Value" "10uF" (id 1) (at 165.1 76.2 0))
-    (property "Footprint" "MATRIX_1.4:CAPACITOR_AE_D5.08mm" (id 2) (at 159.7152 80.01 0)
+    (property "Footprint" "MATRIX_1.4:CAPACITOR_AE_D7.62mm" (id 2) (at 159.7152 80.01 0)
       (effects (font (size 1.27 1.27)) hide)
     )
@@
     (property "Reference" "D411" (id 0) (at 349.25 55.88 90))
     (property "Value" "10A03" (id 1) (at 349.25 58.42 90))
-    (property "Footprint" "MATRIX_1.4:D_5KP_P12.70mm_Horizontal" (id 2) (at 342.9 57.15 0)
+    (property "Footprint" "MATRIX_1.4:DIODE_AXIAL_SMALL_GE" (id 2) (at 342.9 57.15 0)
       (effects (font (size 1.27 1.27)) hide)
     )
@@
   (symbol (lib_id "Device:R") (at 241.3 101.6 180) (unit 1)
     (in_bom yes) (on_board yes)
-    (property "Reference" "R4161" (id 0) (at 247.65 99.06 0))
+    (property "Reference" "R40161" (id 0) (at 247.65 99.06 0))
     (property "Value" "220" (id 1) (at 247.65 101.6 0))
     (property "Footprint" "MATRIX_1.4:RESISTOR_AXIAL_0.5W" (id 2) (at 243.078 101.6 90)
@@
   (symbol (lib_id "Device:R") (at 190.5 152.4 180) (unit 1)
     (in_bom yes) (on_board yes)
-    (property "Reference" "R4144" (id 0) (at 196.85 149.86 0))
+    (property "Reference" "R40144" (id 0) (at 196.85 149.86 0))
     (property "Value" "3.9k" (id 1) (at 196.85 152.4 0))
     (property "Footprint" "MATRIX_1.4:RESISTOR_AXIAL_0.5W" (id 2) (at 192.278 152.4 90)
@@
   (symbol (lib_id "Device:R") (at 327.66 107.95 0) (unit 1)
     (in_bom yes) (on_board yes)
-    (property "Reference" "R4205" (id 0) (at 334.01 105.41 0))
+    (property "Reference" "R4206" (id 0) (at 334.01 105.41 0))
     (property "Value" "0.47" (id 1) (at 334.01 107.95 0))
     (property "Footprint" "MATRIX_1.4:RESISTOR_BLOCK_5W" (id 2) (at 325.882 107.95 90)
@@
   (symbol (lib_id "Device:R") (at 171.45 254 0) (unit 1)
     (in_bom yes) (on_board yes)
-    (property "Reference" "R305" (id 0) (at 177.8 251.46 0))
+    (property "Reference" "R306" (id 0) (at 177.8 251.46 0))
     (property "Value" "10k" (id 1) (at 177.8 254 0))
     (property "Footprint" "MATRIX_1.4:RESISTOR_AXIAL_0.25W" (id 2) (at 169.672 254 90)
@@
   (symbol (lib_id "Device:R") (at 260.35 107.95 180) (unit 1)
     (in_bom yes) (on_board yes)
-    (property "Reference" "R418" (id 0) (at 266.7 105.41 0))
+    (property "Reference" "R4018" (id 0) (at 266.7 105.41 0))
     (property "Value" "10" (id 1) (at 266.7 107.95 0))
     (property "Footprint" "MATRIX_1.4:RESISTOR_AXIAL_2W" (id 2) (at 262.128 107.95 90)
@@
   (symbol (lib_id "Device:R") (at 222.25 171.45 90) (unit 1)
     (in_bom yes) (on_board yes)
-    (property "Reference" "R4151" (id 0) (at 222.25 175.26 90))
+    (property "Reference" "R40151" (id 0) (at 222.25 175.26 90))
     (property "Value" "680" (id 1) (at 222.25 177.8 90))
     (property "Footprint" "MATRIX_1.4:RESISTOR_AXIAL_0.25W" (id 2) (at 222.25 173.228 90)
@@
   (symbol (lib_id "Device:R") (at 171.45 266.7 0) (unit 1)
     (in_bom yes) (on_board yes)
-    (property "Reference" "R306" (id 0) (at 177.8 264.16 0))
+    (property "Reference" "R307" (id 0) (at 177.8 264.16 0))
     (property "Value" "100k" (id 1) (at 177.8 266.7 0))
     (property "Footprint" "MATRIX_1.4:RESISTOR_AXIAL_0.25W" (id 2) (at 169.672 266.7 90)
@@
     (property "Reference" "Q405" (id 0) (at 222.25 144.78 0))
     (property "Value" "MJE350" (id 1) (at 222.25 147.32 0))
-    (property "Footprint" "MATRIX_1.4:TO-225-MIRRORED" (id 2) (at 218.44 148.59 0)
+    (property "Footprint" "MATRIX_1.4:TO-225" (id 2) (at 218.44 148.59 0)
       (effects (font (size 1.27 1.27)) hide)
     )
@@
   (symbol (lib_id "Device:R") (at 228.6 177.8 0) (unit 1)
     (in_bom yes) (on_board yes)
-    (property "Reference" "R4152" (id 0) (at 234.95 175.26 0))
+    (property "Reference" "R40152" (id 0) (at 234.95 175.26 0))
     (property "Value" "100" (id 1) (at 234.95 177.8 0))
     (property "Footprint" "MATRIX_1.4:RESISTOR_AXIAL_0.25W" (id 2) (at 226.822 177.8 90)
@@
   (symbol (lib_id "Device:R") (at 190.5 127 180) (unit 1)
     (in_bom yes) (on_board yes)
-    (property "Reference" "R4142" (id 0) (at 196.85 125.73 0))
+    (property "Reference" "R40142" (id 0) (at 196.85 125.73 0))
     (property "Value" "3.9k" (id 1) (at 196.85 128.27 0))
     (property "Footprint" "MATRIX_1.4:RESISTOR_AXIAL_0.5W" (id 2) (at 192.278 127 90)
@@
   (symbol (lib_id "Device:R") (at 146.05 247.65 90) (unit 1)
     (in_bom yes) (on_board yes)
-    (property "Reference" "R304" (id 0) (at 146.05 251.46 90))
+    (property "Reference" "R305" (id 0) (at 146.05 251.46 90))
     (property "Value" "2.7k" (id 1) (at 146.05 254 90))
     (property "Footprint" "MATRIX_1.4:RESISTOR_AXIAL_0.25W" (id 2) (at 146.05 249.428 90)
@@
   (symbol (lib_id "Device:R") (at 190.5 114.3 180) (unit 1)
     (in_bom yes) (on_board yes)
-    (property "Reference" "R4141" (id 0) (at 196.85 111.76 0))
+    (property "Reference" "R40141" (id 0) (at 196.85 111.76 0))
     (property "Value" "3.9k" (id 1) (at 196.85 114.3 0))
     (property "Footprint" "MATRIX_1.4:RESISTOR_AXIAL_0.5W" (id 2) (at 192.278 114.3 90)
@@
   (symbol (lib_id "Device:R") (at 203.2 266.7 90) (unit 1)
     (in_bom yes) (on_board yes)
-    (property "Reference" "R307" (id 0) (at 203.2 270.51 90))
+    (property "Reference" "R308" (id 0) (at 203.2 270.51 90))
     (property "Value" "3.3k" (id 1) (at 203.2 273.05 90))
     (property "Footprint" "MATRIX_1.4:RESISTOR_AXIAL_0.25W" (id 2) (at 203.2 268.478 90)
@@
   (symbol (lib_id "Device:R") (at 260.35 95.25 180) (unit 1)
     (in_bom yes) (on_board yes)
-    (property "Reference" "R417" (id 0) (at 266.7 92.71 0))
+    (property "Reference" "R4017" (id 0) (at 266.7 92.71 0))
     (property "Value" "10" (id 1) (at 266.7 95.25 0))
     (property "Footprint" "MATRIX_1.4:RESISTOR_AXIAL_2W" (id 2) (at 262.128 95.25 90)
@@
     (property "Reference" "C301" (id 0) (at 165.1 257.81 0))
     (property "Value" "10uF" (id 1) (at 165.1 260.35 0))
-    (property "Footprint" "MATRIX_1.4:CAPACITOR_AE_D5.08mm" (id 2) (at 159.7152 264.16 0)
+    (property "Footprint" "MATRIX_1.4:CAPACITOR_AE_D7.62mm" (id 2) (at 159.7152 264.16 0)
       (effects (font (size 1.27 1.27)) hide)
     )
@@
   (symbol (lib_id "Device:R") (at 190.5 139.7 180) (unit 1)
     (in_bom yes) (on_board yes)
-    (property "Reference" "R4143" (id 0) (at 196.85 137.16 0))
+    (property "Reference" "R40143" (id 0) (at 196.85 137.16 0))
     (property "Value" "3.9k" (id 1) (at 196.85 139.7 0))
     (property "Footprint" "MATRIX_1.4:RESISTOR_AXIAL_0.5W" (id 2) (at 192.278 139.7 90)
@@
     (property "Reference" "R514" (id 0) (at 165.1 200.66 0))
     (property "Value" "100k" (id 1) (at 165.1 203.2 0))
-    (property "Footprint" "MATRIX_1.4:RESISTOR_AXIAL_0.5W" (id 2) (at 156.972 203.2 90)
+    (property "Footprint" "MATRIX_1.4:RESISTOR_AXIAL_0.25W" (id 2) (at 156.972 203.2 90)
       (effects (font (size 1.27 1.27)) hide)
     )
@@
   (symbol (lib_id "Device:R") (at 133.35 260.35 90) (unit 1)
     (in_bom yes) (on_board yes)
-    (property "Reference" "R303" (id 0) (at 133.35 264.16 90))
+    (property "Reference" "R304" (id 0) (at 133.35 264.16 90))
     (property "Value" "10k" (id 1) (at 133.35 266.7 90))
     (property "Footprint" "MATRIX_1.4:RESISTOR_AXIAL_0.25W" (id 2) (at 133.35 262.128 90)
@@
     (property "Reference" "C503" (id 0) (at 292.1 226.06 0))
     (property "Value" "1uF" (id 1) (at 292.1 228.6 0))
-    (property "Footprint" "MATRIX_1.4:CAPACITOR_AE_D5.08mm" (id 2) (at 286.7152 232.41 0)
+    (property "Footprint" "MATRIX_1.4:CAPACITOR_AE_D7.62mm" (id 2) (at 286.7152 232.41 0)
       (effects (font (size 1.27 1.27)) hide)
     )
@@
   (symbol (lib_id "MATRIX_1.4:RAYEX-L90A") (at 373.38 209.55 0) (unit 1)
     (in_bom yes) (on_board yes)
-    (property "Reference" "S501" (id 0) (at 387.35 209.55 0))
+    (property "Reference" "S1" (id 0) (at 387.35 209.55 0))
     (property "Value" "sw1 ON" (id 1) (at 384.81 210.8199 0)
       (effects (font (size 1.27 1.27)) (justify left) hide)
     )
-    (property "Footprint" "MATRIX_1.4:Relay_SPDT_RAYEX-L90" (id 2) (at 384.81 210.82 0)
+    (property "Footprint" "Relay_THT:Relay_SPST_RAYEX-L90A" (id 2) (at 384.81 210.82 0)
       (effects (font (size 1.27 1.27)) (justify left) hide)
     )
