File: MATRIX-1.4-IV-T13-H-DEV-1/MATRIX-1.4-IV-T13-H-DEV-1.kicad_sch (KiCad schematic)
At the start: 214 parts, among them Q401 2N5551, Q402 2N5551, Q403 MJE340, Q404 MJE350, Q405 MJE350, Q406 MJE350, Q407 MJE340, Q408 MJE350, Q409 MJE340, Q410 MJE15032, Q411 MJE15033, Q412 2SC5200, Q413 2SA1943, Q4141 2SC5200, Q41410 2SC5200, Q4142 2SC5200, Q4143 2SC5200, Q4144 2SC5200, Q4145 2SC5200, Q4146 2SC5200, Q4147 2SC5200, Q4148 2SC5200, Q4149 2SC5200, Q4151 2SA1943, Q41510 2SA1943, Q4152 2SA1943, Q4153 2SA1943, Q4154 2SA1943, Q4155 2SA1943, Q4156 2SA1943, Q4157 2SA1943, Q4158 2SA1943, Q4159 2SA1943, Q501 2N5401, Q502 2N5551, Q503 2N5401, Q504 2N5551, Q505 2N5551, Q506 2N5401, Q507 2N5551, Q508 2N5551, Q509 TIP41C, Q601 2N5551, Q602 2N5401, Q603 2N5401, Q604 2N5401, Q605 2N5401, Q606 2N5551, Q701 2N5401, Q702 2N5551, Q703 2N5551, Q704 2N5551, Q705 2N5551, Q706 2N5401

Commit message: Routine Update Tue Jun 14 09:06:30 AM WIB 2022
Parts:
- renumbered C900 to C404, C404 to C405, C405 to C406, C406 to C407
Changed lines of the file:
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@@
   (symbol (lib_id "Device:C") (at 133.35 133.35 180) (unit 1)
     (in_bom yes) (on_board yes)
-    (property "Reference" "C404" (id 0) (at 139.7 130.81 0))
+    (property "Reference" "C405" (id 0) (at 139.7 130.81 0))
     (property "Value" "0.1uF" (id 1) (at 139.7 133.35 0))
     (property "Footprint" "MATRIX_1.4:CAPACITOR_MPF_STD" (id 2) (at 132.3848 129.54 0)
@@
   (symbol (lib_id "Device:C") (at 127 158.75 90) (unit 1)
     (in_bom yes) (on_board yes)
-    (property "Reference" "C405" (id 0) (at 127 149.86 90))
+    (property "Reference" "C406" (id 0) (at 127 149.86 90))
     (property "Value" "47pF" (id 1) (at 127 152.4 90))
     (property "Footprint" "MATRIX_1.4:CAPACITOR_CERAMIC_STD" (id 2) (at 130.81 157.7848 0)
@@
   (symbol (lib_id "Device:C") (at 374.65 120.65 180) (unit 1)
     (in_bom yes) (on_board yes)
-    (property "Reference" "C406" (id 0) (at 381 118.11 0))
+    (property "Reference" "C407" (id 0) (at 381 118.11 0))
     (property "Value" "0.1uF" (id 1) (at 381 120.65 0))
     (property "Footprint" "MATRIX_1.4:CAPACITOR_MPF_STD" (id 2) (at 373.6848 116.84 0)
@@
   (symbol (lib_id "Device:C") (at 88.9 50.8 90) (unit 1)
     (in_bom yes) (on_board yes)
-    (property "Reference" "C900" (id 0) (at 88.9 54.61 90))
+    (property "Reference" "C404" (id 0) (at 88.9 54.61 90))
     (property "Value" "47pF" (id 1) (at 88.9 57.15 90))
     (property "Footprint" "MATRIX_1.4:CAPACITOR_CERAMIC_STD" (id 2) (at 92.71 49.8348 0)

Commit message: Routine Update Sat Jun 18 06:31:12 PM WIB 2022
Parts:
- added C601, C701: 470pF, MATRIX_1.4:CAPACITOR_CERAMIC_STD, symbol Device:C
- added Q607: BF423, MATRIX_1.4:TO-92-EBC, symbol MATRIX_1.4:Q_PNP_CBE
- added Q707: BF422, MATRIX_1.4:TO-92-EBC, symbol MATRIX_1.4:Q_NPN_CBE
- added R611, R711: 10k, MATRIX_1.4:RESISTOR_AXIAL_0.25W, symbol Device:R
- added R612, R712: 10k, MATRIX_1.4:RESISTOR_AXIAL_0.5W, symbol Device:R
- D605: value 1N4738 -> 1N4742; Spice_Model 1N4738 -> 1N4742
- D705: value 1N4738 -> 1N4742
Connections:
- net +60V: now also Q604.1 (C), R611.1
- net -60V: now also Q704.1 (C), R711.1
- net VSHN: now also Q707.3 (E), R612.1
- net VSHP: now also Q607.3 (E), R712.2
- net at D704.2 (K), R706.1: no longer Q704.1 (C)
- net at D604.1 (A), R606.1: no longer Q604.1 (C)
- net at R609.1: now also D607.1 (A), Q606.2 (B), R610.2, C601.2; no longer Q605.1 (C)
- net at D707.2 (K), Q706.2 (B), R709.1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: now also C701.2
- net at D708.1 (A), Q706.1 (C): now also C701.1
- net at D608.2 (K), Q606.1 (C): now also C601.1
- new net: Q707.1 (C), R712.1
- new net: Q707.2 (B), R711.2
- new net: Q607.2 (B), R611.2
- new net: Q607.1 (C), R612.2
- new net: Q605.1 (C), R609.2
Other:
- moved on the sheet: C407, C501, C503, C504, D411, D412, D507, D508, D511, D512, D513, D514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

Commit message: Routine Update Sat Jun 18 06:40:31 PM WIB 2022
Other:
- note added: "> MAIN AMPLIFIER BLOCK > STEPPER > PROTECTOR"
- moved on the sheet: C501, C502, C503, C504, D501, D502, D503, D504, D505, D506, D507, D508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
