File: MATRIX-1.4-IV-T13-TD-DEV-1/MATRIX-1.4-IV-T13-TD-DEV-1.kicad_sch (KiCad schematic)
At the start: 155 parts, among them Q401 MPSA42, Q402 MPSA42, Q403 MPSA92, Q404 MPSA92, Q405 MJE340, Q406 MJE350, Q407 MJE350, Q408 MJE340, Q409 MJE15032, Q410 MJE15033, Q411 2SC5200, Q412 2SA1943, Q4131 2SC5200, Q4132 2SC5200, Q4133 2SC5200, Q4134 2SC5200, Q4135 2SC5200, Q4136 2SC5200, Q4141 2SA1943, Q4142 2SA1943, Q4143 2SA1943, Q4144 2SA1943, Q4145 2SA1943, Q4146 2SA1943, Q601 2N5401, Q602 MJE15032, Q603 2SC5200, Q604 2N5401, Q605 2N5401, Q606 2N5401, Q607 2N5401, Q608 2N5401, Q609 2N5401, Q701 2N5551, Q702 MJE15033, Q703 2SA1943, Q704 2N5551, Q705 2N5551, Q706 2N5551, Q707 2N5551, Q708 2N5551, Q709 2N5551

Commit message: Routine Update Wed Jul 27 08:27:36 PM WIB 2022
Parts:
- removed D707: 1N4746, MATRIX_1.4:DIODE_AXIAL_SMALL_SI, symbol MATRIX_1.4:D_Zener
- added C603, C703: 4.7uF, MATRIX_1.4:CAPACITOR_AE_D10mm, symbol Device:C_Polarized
- added C604, C704: 47uF, MATRIX_1.4:CAPACITOR_AE_D10mm, symbol Device:C_Polarized
- added D708: 1N4749, MATRIX_1.4:DIODE_AXIAL_SMALL_SI, symbol MATRIX_1.4:D_Zener
- added Q603: MJE15032, MATRIX_1.4:TO-220-MIRRORED, symbol MATRIX_1.4:Q_NPN_CBE
- added Q611: 2N5401, MATRIX_1.4:TO-92-EBC, symbol MATRIX_1.4:Q_PNP_CBE
- added Q612: MJE340, MATRIX_1.4:TO-225, symbol MATRIX_1.4:Q_NPN_CBE
- added Q703: MJE15033, MATRIX_1.4:TO-220-MIRRORED, symbol MATRIX_1.4:Q_PNP_CBE
- added Q711: 2N5551, MATRIX_1.4:TO-92-EBC, symbol MATRIX_1.4:Q_NPN_CBE
- added Q712: MJE350, MATRIX_1.4:TO-225, symbol MATRIX_1.4:Q_PNP_CBE
- added R605, R705: 56, MATRIX_1.4:RESISTOR_AXIAL_0.5W, symbol Device:R
- added R614, R714: 100k, MATRIX_1.4:RESISTOR_AXIAL_0.5W, symbol Device:R
- C602, C702: value 68pF -> 12pF
- D608: renamed from D607; value 1N4746 -> 1N4749; Spice_Model 1N4746 -> 1N4749
- Q602: value MJE15032 -> MJE340; footprint MATRIX_1.4:TO-220-MIRRORED -> MATRIX_1.4:TO-225; Spice_Model MJE15032 -> MJE340
- Q608: renamed from Q607; Spice_Model 2N5401 -> MJE350
- Q702: value MJE15033 -> MJE350; footprint MATRIX_1.4:TO-220-MIRRORED -> MATRIX_1.4:TO-225; Spice_Model MJE15033 -> MJE350
- R601, R701: value 1.2k -> 12k
- R602, R603, R702, R703: value 22k -> 120k
- R604, R704: value 120 -> 1.5k
- R608: renamed from R607; value 15k -> 2.7k
- R610: renamed from R609; value 15k -> 2.7k
- R612: renamed from R611; value 15k -> 2.7k
- R708: renamed from R707; value 15k -> 2.7k
- R710: renamed from R709; value 15k -> 2.7k
- R712: renamed from R711; value 15k -> 2.7k
- renumbered C603 to C605, C604 to C606, C703 to C705, C704 to C706, D608 to D607, D708 to D707, Q603 to Q604, Q604 to Q605, Q605 to Q606, Q606 to Q607, Q608 to Q609, Q609 to Q610, Q703 to Q704, Q704 to Q705, Q705 to Q706, Q706 to Q707, Q707 to Q708, Q708 to Q709, Q709 to Q710, R605 to R606, R606 to R607, R608 to R609, R610 to R611, R612 to R613, R613 to R615, R705 to R706, R706 to R707, R708 to R709, R710 to R711, R712 to R713, R713 to R715
Connections:
- net +120V: now also C603.1, C604.1, Q603.1 (C)
- net -120V: now also C703.2, C704.2, D708.1 (A), Q703.1 (C)
- net 0: now also Q612.3 (E), Q712.3 (E), R614.2, R714.1; no longer Q608.1 (C), Q708.1 (C), R608.2, R610.2, R612.2, R708.2, R710.2, R712.1
- net VSAVN: now also R705.1
- net VSAVP: now also R605.2
- net VSGZP: no longer D608.1 (A)
- net at Q702.3 (E), R704.2: now also Q703.2 (B); no longer Q704.2 (B)
- net at D707.1 (A), Q709.2 (B): now also R712.1; no longer R712.2
- net VSTAN: now reaches D706.2 (K), D707.2 (K), Q705.1 (C)
- net VSTAP: now reaches D606.1 (A), D607.1 (A), Q605.1 (C)
- net at Q602.3 (E), R604.1: now also Q603.2 (B); no longer Q604.2 (B)
- new net: Q603.3 (E), Q604.2 (B), R605.1
- new net: Q703.3 (E), Q704.2 (B), R705.2
- new net: Q711.1 (C), Q712.2 (B)
- new net: C703.1, D708.2 (K), Q711.2 (B), R714.2
- new net: C603.2, D608.1 (A), Q611.2 (B), R614.1
- new net: Q611.1 (C), Q612.2 (B)
- new net VSGSPN: C704.1, Q708.1 (C), Q711.3 (E), Q712.1 (C), R708.2, R710.2, R712.2
- new net VSGSPP: C604.2, Q608.1 (C), Q611.3 (E), Q612.1 (C), R608.2, R610.2, R612.2
Other:
- moved on the sheet: C406, C601, C602, C605, C606, C701, C702, C705, C706, D402, D403, D601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

Commit message: Routine Update Thu Jul 28 08:53:49 PM WIB 2022
Parts:
- C602, C702: value 12pF -> 22pF
Changed lines of the file:
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@@
     (in_bom yes) (on_board yes)
     (property "Reference" "C602" (id 0) (at 190.5 29.21 0))
-    (property "Value" "12pF" (id 1) (at 190.5 31.75 0))
+    (property "Value" "22pF" (id 1) (at 190.5 31.75 0))
     (property "Footprint" "MATRIX_1.4:CAPACITOR_CERAMIC_LEAD_PITCH_7.62mm" (id 2) (at 183.1848 27.94 0)
       (effects (font (size 1.27 1.27)) hide)
@@
     (in_bom yes) (on_board yes)
     (property "Reference" "C702" (id 0) (at 190.5 207.01 0))
-    (property "Value" "12pF" (id 1) (at 190.5 209.55 0))
+    (property "Value" "22pF" (id 1) (at 190.5 209.55 0))
     (property "Footprint" "MATRIX_1.4:CAPACITOR_CERAMIC_LEAD_PITCH_7.62mm" (id 2) (at 183.1848 205.74 0)
       (effects (font (size 1.27 1.27)) hide)

Commit message: Routine Update Fri Jul 29 01:06:43 PM WIB 2022
Parts:
- R608, R610, R612, R708, R710, R712: value 2.7k -> 1.5k
- R609, R613, R614, R702, R703, R709, R713, R714: footprint MATRIX_1.4:RESISTOR_AXIAL_0.5W -> MATRIX_1.4:RESISTOR_AXIAL_0.25W; Wattage 0.5W -> 0.25W
Connections:
- net VASDEP: no longer names the net of Q406.3 (E), R4091.2, R4092.2
