File: MATRIX-1.4-IV-T13-TD-DEV-1/ANALYSIS-MATRIX-1.4-IV-T13-TD-DEV-1.kicad_sch (KiCad schematic)
At the start: 6 parts

Commit message: Routine Update Sun Jul 10 09:42:39 PM WIB 2022
Connections:
- net P_OUTPUT renamed VPOUT
