File: MATRIX-1.4-IV-T13-TD-DEV-1/ANALYSIS-MATRIX-1.4-IV-T13-TD-DEV-1.kicad_sch (KiCad schematic)
At the start: 6 parts

Commit message: Routine Update Sat Jul 23 04:17:04 PM WIB 2022
Parts:
- V11, V12: value 120V DC -> DC 120V
- V31, V32: value 15V DC -> DC 15V
Other:
- note added: "* Transient analysis directive for 1KHz with input at 1.41Vp * To apply the directive, please uncomment the line below. .tran 0.1u 1m .fourier 1k v(vmout)"
- note removed: "* Transient analysis directive for 1KHz with input at 1.41Vp * To apply the directive, please uncomment the line below. *.tran 1u 22m 20m"
