File: MATRIX-1.4-IV-T13-TD-DEV-1/ANALYSIS-MATRIX-1.4-IV-T13-TD-DEV-1.kicad_sch (KiCad schematic)
At the start: 6 parts

Commit message: Routine Update Mon Jul 25 04:47:29 PM WIB 2022
Other:
- note added: "* Transient analysis directive for 1KHz with input at 1.41Vp * To apply the directive, please uncomment the line below. *.tran 0.1u 1m *.fourier 1k v(vmout)"
- note removed: "* Transient analysis directive for 1KHz with input at 1.41Vp * To apply the directive, please uncomment the line below. .tran 0.1u 1m .fourier 1k v(vmout)"
Changed lines of the file:
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@@
     (effects (font (size 1.905 1.905)) (justify left bottom))
   )
-  (text "* Transient analysis directive for 1KHz with input at 1.41Vp\n* To apply the directive, please uncomment the line below.\n.tran 0.1u 1m\n.fourier 1k v(vmout)"
+  (text "* Transient analysis directive for 1KHz with input at 1.41Vp\n* To apply the directive, please uncomment the line below.\n*.tran 0.1u 1m\n*.fourier 1k v(vmout)"
     (at 38.1 148.59 0)
     (effects (font (size 1.27 1.27)) (justify left bottom))
@@
     )
     (path "/00000000-0000-0000-0000-000060b22bae/84b8f5d6-1be1-49a2-9cad-ba2ca688ac42"
-      (reference "C602") (unit 1) (value "100pF") (footprint "MATRIX_1.4:CAPACITOR_CERAMIC_LEAD_PITCH_7.62mm")
+      (reference "C602") (unit 1) (value "68pF") (footprint "MATRIX_1.4:CAPACITOR_CERAMIC_LEAD_PITCH_7.62mm")
     )
     (path "/00000000-0000-0000-0000-000060b22bae/aa9aa012-4a84-4b4f-ad77-f4dabe72ed54"
@@
     )
     (path "/00000000-0000-0000-0000-000060b22bae/ebec87b1-b202-4bbf-877d-3d341636a6e1"
-      (reference "C702") (unit 1) (value "100pF") (footprint "MATRIX_1.4:CAPACITOR_CERAMIC_LEAD_PITCH_7.62mm")
+      (reference "C702") (unit 1) (value "68pF") (footprint "MATRIX_1.4:CAPACITOR_CERAMIC_LEAD_PITCH_7.62mm")
     )
     (path "/00000000-0000-0000-0000-000060b22bae/d4af786d-ce6a-4fae-b270-4fd52c1f0fed"

Commit message: Routine Update Sat Jul 30 08:21:57 AM WIB 2022
Parts:
- removed V31, V32: DC 15V, symbol pspice:VSOURCE
- renumbered Rdummy1 to R901
Connections:
- net POWER-AMP/+120V renamed +120V
- net POWER-AMP/-120V renamed -120V
Other:
- sheet POWER-AMP ports: added none; removed +120V, +15V, -120V, -15V
- moved on the sheet: R901, V11, V12, V20
