File: MATRIX-1.4-IV-T13-TD-DEV-3/MATRIX-1.4-IV-T13-TD-DEV-3.kicad_sch (KiCad schematic)
At the start: 181 parts

Commit message: Routine Update Sun Jul 31 03:58:44 PM WIB 2022
Parts:
- C401: value (none) -> 10uF; footprint (none) -> MATRIX_1.4:CAPACITOR_AE_D7.62mm
- C402: value (none) -> 220pF; footprint (none) -> MATRIX_1.4:CAPACITOR_CERAMIC_LEAD_PITCH_7.5mm
- C403: value (none) -> 220uF; footprint (none) -> MATRIX_1.4:CAPACITOR_AE_D10mm
- C404: value (none) -> 220pF; footprint (none) -> MATRIX_1.4:CAPACITOR_CERAMIC_LEAD_PITCH_7.62mm
- C405, C406, C407, C409: value (none) -> 0.1uF; footprint (none) -> MATRIX_1.4:0.1uF_250V_Vishay_Roederstein_MKT_1822
- C408, C410: value (none) -> 10uF; footprint (none) -> MATRIX_1.4:CAPACITOR_AE_D10mm
- C601, C603, C701, C703: value (none) -> 4.7uF; footprint (none) -> MATRIX_1.4:CAPACITOR_AE_D10mm
- C602, C702: value (none) -> 33pF; footprint (none) -> MATRIX_1.4:CAPACITOR_CERAMIC_LEAD_PITCH_7.62mm
- C604, C704: value (none) -> 47uF; footprint (none) -> MATRIX_1.4:CAPACITOR_AE_D10mm
- C605, C705: value (none) -> 2200pF; footprint (none) -> MATRIX_1.4:0.0022uF_400V_Vishay_Roederstein_MKT_1822
- C606: value (none) -> 1uF; footprint (none) -> MATRIX_1.4:0.1uF_250V_Vishay_Roederstein_MKT_1822
- C706: value (none) -> 1uF; footprint (none) -> MATRIX_1.4:1uF_250V_Vishay_Roederstein_MKT_1822
- D401: value (none) -> 1N4732; footprint (none) -> MATRIX_1.4:DIODE_AXIAL_SMALL_SI
- D402, D403, D604, D605, D609, D704, D705, D709: value (none) -> MURF1560; footprint (none) -> MATRIX_1.4:DIODE_AXIAL_SMALL_GE
- D601, D701: value (none) -> 1N4007; footprint (none) -> MATRIX_1.4:DIODE_AXIAL_SMALL_SI
- D602, D702: value (none) -> BAV21; footprint (none) -> MATRIX_1.4:DIODE_AXIAL_SMALL_SI
- D603, D703: value (none) -> 1N4734; footprint (none) -> MATRIX_1.4:DIODE_AXIAL_SMALL_SI
- D606, D607, D706, D707: value (none) -> BAV21; footprint (none) -> MATRIX_1.4:DIODE_AXIAL_SMALL_GE
- D608, D708: value (none) -> 1N4749; footprint (none) -> MATRIX_1.4:DIODE_AXIAL_SMALL_SI
- L401: value (none) -> 1uH; footprint (none) -> MATRIX_1.4:INDUCTOR_AIR_CORE_3uH_D600mils_L750mils
- L601, L701: value (none) -> 10uH; footprint (none) -> MATRIX_1.4:TOROIDAL_INDUCTOR_0077083A7
- Q401, Q402: value (none) -> MPSA42; footprint (none) -> MATRIX_1.4:TO-92-EBC
- Q403, Q404: value (none) -> MPSA92; footprint (none) -> MATRIX_1.4:TO-92-EBC
- Q405, Q408, Q602, Q614: value (none) -> MJE340; footprint (none) -> MATRIX_1.4:TO-225
- Q406, Q407, Q702, Q714: value (none) -> MJE350; footprint (none) -> MATRIX_1.4:TO-225
- Q409, Q603: value (none) -> MJE15032; footprint (none) -> MATRIX_1.4:TO-220-MIRRORED
- Q410, Q703: value (none) -> MJE15033; footprint (none) -> MATRIX_1.4:TO-220-MIRRORED
- Q411, Q4131, Q4132, Q4133, Q4134, Q4135, Q4136, Q604: value (none) -> 2SC5200; footprint (none) -> MATRIX_1.4:TO-264-MIRRORED
- Q412, Q4141, Q4142, Q4143, Q4144, Q4145, Q4146, Q704: value (none) -> 2SA1943; footprint (none) -> MATRIX_1.4:TO-264-MIRRORED
- Q601, Q605, Q608, Q609, Q611, Q612, Q613, Q706, Q707, Q710: value (none) -> 2N5401; footprint (none) -> MATRIX_1.4:TO-92-EBC
- Q606, Q607, Q610, Q701, Q705, Q708, Q709, Q711, Q712, Q713: value (none) -> 2N5551; footprint (none) -> MATRIX_1.4:TO-92-EBC
- R401, R404: value (none) -> 180; footprint (none) -> MATRIX_1.4:RESISTOR_AXIAL_0.25W
- R4021, R4031, R613: value (none) -> 15k; footprint (none) -> MATRIX_1.4:RESISTOR_AXIAL_0.5W
- R4022, R4032: value (none) -> 270k; footprint (none) -> MATRIX_1.4:RESISTOR_AXIAL_0.5W
- R4051, R4061: value (none) -> 56; footprint (none) -> MATRIX_1.4:RESISTOR_AXIAL_0.25W
- R4052, R4062, R4081, R4141: value (none) -> 470; footprint (none) -> MATRIX_1.4:RESISTOR_AXIAL_0.25W
- R4071, R4072, R4073, R4074: value (none) -> 56k; footprint (none) -> MATRIX_1.4:RESISTOR_AXIAL_0.25W
- R4082, R4142: value (none) -> 47k; footprint (none) -> MATRIX_1.4:RESISTOR_AXIAL_0.25W
- R4091, R607, R707: value (none) -> 150; footprint (none) -> MATRIX_1.4:RESISTOR_AXIAL_0.25W
- R4092: value (none) -> 820; footprint (none) -> MATRIX_1.4:RESISTOR_AXIAL_0.25W
- R410: value (none) -> 1.2k; footprint (none) -> MATRIX_1.4:RESISTOR_AXIAL_0.25W
- R411, R412: value (none) -> 390; footprint (none) -> MATRIX_1.4:RESISTOR_AXIAL_0.25W
- R413: value (none) -> 2.2k; footprint (none) -> MATRIX_1.4:RESISTOR_AXIAL_0.25W
- R4151: value (none) -> 120; footprint (none) -> MATRIX_1.4:RESISTOR_AXIAL_0.5W
- R416, R417: value (none) -> 5.6; footprint (none) -> MATRIX_1.4:RESISTOR_BLOCK_5W
- R4181, R4182, R4183, R4184, R4185, R4186, R4191, R4192, R4193, R4194, R4195, R4196: value (none) -> 0.33; footprint (none) -> MATRIX_1.4:RESISTOR_BLOCK_5W
- R420: value (none) -> 10; footprint (none) -> MATRIX_1.4:RESISTOR_BLOCK_5W
- R601, R701: value (none) -> 12k; footprint (none) -> MATRIX_1.4:RESISTOR_AXIAL_0.5W
- R602, R603: value (none) -> 120k; footprint (none) -> MATRIX_1.4:RESISTOR_AXIAL_0.5W
- R604, R704: value (none) -> 1.5k; footprint (none) -> MATRIX_1.4:RESISTOR_AXIAL_0.5W
- R605, R705: value (none) -> 56; footprint (none) -> MATRIX_1.4:RESISTOR_AXIAL_0.5W
- R606, R706: value (none) -> 1; footprint (none) -> MATRIX_1.4:RESISTOR_BLOCK_5W
- R608, R609, R610, R611, R612, R615, R708, R709, R710, R712, R715: value (none) -> 2.7k; footprint (none) -> MATRIX_1.4:RESISTOR_AXIAL_0.5W
- R614: value (none) -> 2.7k; footprint (none) -> MATRIX_1.4:RESISTOR_AXIAL_0.25W; Wattage 0.25W -> 0.5W
- R616, R716: value (none) -> 4.7; footprint (none) -> MATRIX_1.4:RESISTOR_AXIAL_0.5W
- R617, R717: value (none) -> 27k; footprint (none) -> MATRIX_1.4:RESISTOR_AXIAL_0.25W
- R618, R718: value (none) -> 100k; footprint (none) -> MATRIX_1.4:RESISTOR_AXIAL_0.25W
- R619, R719: value (none) -> 680; footprint (none) -> MATRIX_1.4:RESISTOR_AXIAL_0.5W
- R702, R703: value (none) -> 120k; footprint (none) -> MATRIX_1.4:RESISTOR_AXIAL_0.25W
- R711, R714: value (none) -> 2.7k; footprint (none) -> MATRIX_1.4:RESISTOR_AXIAL_0.25W
- R713: value (none) -> 15k; footprint (none) -> MATRIX_1.4:RESISTOR_AXIAL_0.25W
- RT401: value (none) -> 5k; footprint (none) -> MATRIX_1.4:RESISTOR_ROUND_TRIMPOT_STD
- XQ6011, XQ6012: value (none) -> IRF9640; footprint (none) -> MATRIX_1.4:TO-220-MIRRORED
- XQ7011, XQ7012: value (none) -> IRF640; footprint (none) -> MATRIX_1.4:TO-220-MIRRORED
Other:
- moved on the sheet: C705, D709, L701, R719
