File: MATRIX-1.4-IV-T13-TD-DEV-3/MATRIX-1.4-IV-T13-TD-DEV-3.kicad_sch (KiCad schematic)
At the start: 181 parts, among them Q401 MPSA42, Q402 MPSA42, Q403 MPSA92, Q404 MPSA92, Q405 MJE340, Q406 MJE350, Q407 MJE350, Q408 MJE340, Q409 MJE15032, Q410 MJE15033, Q411 2SC5200, Q412 2SA1943, Q4131 2SC5200, Q4132 2SC5200, Q4133 2SC5200, Q4134 2SC5200, Q4135 2SC5200, Q4136 2SC5200, Q4141 2SA1943, Q4142 2SA1943, Q4143 2SA1943, Q4144 2SA1943, Q4145 2SA1943, Q4146 2SA1943, Q601 2N5401, Q602 MJE340, Q603 MJE15032, Q604 2SC5200, Q605 2N5401, Q606 2N5551, Q607 2N5551, Q608 2N5401, Q609 2N5401, Q610 2N5551, Q611 2N5401, Q612 2N5401, Q613 2N5401, Q614 MJE340, Q701 2N5551, Q702 MJE350, Q703 MJE15033, Q704 2SA1943, Q705 2N5551, Q706 2N5401, Q707 2N5401, Q708 2N5551, Q709 2N5551, Q710 2N5401, Q711 2N5551, Q712 2N5551, Q713 2N5551, Q714 MJE350

Commit message: Routine Update Sun Jul 31 07:24:30 PM WIB 2022
Parts:
- R601, R602, R603, R604, R608, R609, R610, R611, R612, R613, R615, R701, R704, R708, R709, R710, R712, R715: footprint MATRIX_1.4:RESISTOR_AXIAL_0.5W -> MATRIX_1.4:RESISTOR_AXIAL_0.25W; Wattage 0.5W -> 0.25W
- R605: Wattage 5W -> 0.5W
- R614: Wattage 0.5W -> 0.25W

Commit message: Routine Update Tue Aug  2 09:19:02 AM WIB 2022
Parts:
- removed C401: 10uF, MATRIX_1.4:CAPACITOR_AE_D7.62mm, symbol Device:C_Polarized
- removed C402: 220pF, MATRIX_1.4:CAPACITOR_CERAMIC_LEAD_PITCH_7.5mm, symbol Device:C
- removed C403: 220uF, MATRIX_1.4:CAPACITOR_AE_D10mm, symbol Device:C_Polarized
- removed C404: 220pF, MATRIX_1.4:CAPACITOR_CERAMIC_LEAD_PITCH_7.62mm, symbol Device:C
- removed C405, C406, C407, C409: 0.1uF, MATRIX_1.4:0.1uF_250V_Vishay_Roederstein_MKT_1822, symbol Device:C
- removed C408, C410: 10uF, MATRIX_1.4:CAPACITOR_AE_D10mm, symbol Device:C_Polarized
- removed C601, C603, C701, C703: 4.7uF, MATRIX_1.4:CAPACITOR_AE_D10mm, symbol Device:C_Polarized
- removed C602, C702: 33pF, MATRIX_1.4:CAPACITOR_CERAMIC_LEAD_PITCH_7.62mm, symbol Device:C
- removed C604, C704: 47uF, MATRIX_1.4:CAPACITOR_AE_D10mm, symbol Device:C_Polarized
- removed C605, C705: 2200pF, MATRIX_1.4:0.0022uF_400V_Vishay_Roederstein_MKT_1822, symbol Device:C
- removed C606: 1uF, MATRIX_1.4:0.1uF_250V_Vishay_Roederstein_MKT_1822, symbol Device:C
- removed C706: 1uF, MATRIX_1.4:1uF_250V_Vishay_Roederstein_MKT_1822, symbol Device:C
- removed D401: 1N4732, MATRIX_1.4:DIODE_AXIAL_SMALL_SI, symbol MATRIX_1.4:D_Zener
- removed D402, D403, D604, D605, D609, D704, D705, D709: MURF1560, MATRIX_1.4:DIODE_AXIAL_SMALL_GE, symbol MATRIX_1.4:D
- removed D601, D701: 1N4007, MATRIX_1.4:DIODE_AXIAL_SMALL_SI, symbol MATRIX_1.4:D
- removed D602, D702: BAV21, MATRIX_1.4:DIODE_AXIAL_SMALL_SI, symbol MATRIX_1.4:D
- removed D603, D703: 1N4734, MATRIX_1.4:DIODE_AXIAL_SMALL_SI, symbol MATRIX_1.4:D_Zener
- removed D606, D607, D706, D707: BAV21, MATRIX_1.4:DIODE_AXIAL_SMALL_GE, symbol MATRIX_1.4:D
- removed D608, D708: 1N4749, MATRIX_1.4:DIODE_AXIAL_SMALL_SI, symbol MATRIX_1.4:D_Zener
- removed L401: 1uH, MATRIX_1.4:INDUCTOR_AIR_CORE_3uH_D600mils_L750mils, symbol Device:L_Small
- removed L601, L701: 10uH, MATRIX_1.4:TOROIDAL_INDUCTOR_0077083A7, symbol Device:L_Ferrite
- removed Q401, Q402: MPSA42, MATRIX_1.4:TO-92-EBC, symbol MATRIX_1.4:Q_NPN_CBE
- removed Q403, Q404: MPSA92, MATRIX_1.4:TO-92-EBC, symbol MATRIX_1.4:Q_PNP_CBE
- removed Q405, Q408, Q602, Q614: MJE340, MATRIX_1.4:TO-225, symbol MATRIX_1.4:Q_NPN_CBE
- removed Q406, Q407, Q702, Q714: MJE350, MATRIX_1.4:TO-225, symbol MATRIX_1.4:Q_PNP_CBE
- removed Q409, Q603: MJE15032, MATRIX_1.4:TO-220-MIRRORED, symbol MATRIX_1.4:Q_NPN_CBE
- removed Q410, Q703: MJE15033, MATRIX_1.4:TO-220-MIRRORED, symbol MATRIX_1.4:Q_PNP_CBE
- removed Q411, Q4131, Q4132, Q4133, Q4134, Q4135, Q4136, Q604: 2SC5200, MATRIX_1.4:TO-264-MIRRORED, symbol MATRIX_1.4:Q_NPN_CBE
- removed Q412, Q4141, Q4142, Q4143, Q4144, Q4145, Q4146, Q704: 2SA1943, MATRIX_1.4:TO-264-MIRRORED, symbol MATRIX_1.4:Q_PNP_CBE
- removed Q601, Q605, Q608, Q609, Q611, Q612, Q613, Q706, Q707, Q710: 2N5401, MATRIX_1.4:TO-92-EBC, symbol MATRIX_1.4:Q_PNP_CBE
- removed Q606, Q607, Q610, Q701, Q705, Q708, Q709, Q711, Q712, Q713: 2N5551, MATRIX_1.4:TO-92-EBC, symbol MATRIX_1.4:Q_NPN_CBE
- removed R401, R404: 180, MATRIX_1.4:RESISTOR_AXIAL_0.25W, symbol Device:R
- removed R4021, R4031: 15k, MATRIX_1.4:RESISTOR_AXIAL_0.5W, symbol Device:R
- removed R4022, R4032: 270k, MATRIX_1.4:RESISTOR_AXIAL_0.5W, symbol Device:R
- removed R4051, R4061: 56, MATRIX_1.4:RESISTOR_AXIAL_0.25W, symbol Device:R
- removed R4052, R4062, R4081, R4141: 470, MATRIX_1.4:RESISTOR_AXIAL_0.25W, symbol Device:R
- removed R4071, R4072, R4073, R4074: 56k, MATRIX_1.4:RESISTOR_AXIAL_0.25W, symbol Device:R
- removed R4082, R4142: 47k, MATRIX_1.4:RESISTOR_AXIAL_0.25W, symbol Device:R
- removed R4091, R607, R707: 150, MATRIX_1.4:RESISTOR_AXIAL_0.25W, symbol Device:R
- removed R4092: 820, MATRIX_1.4:RESISTOR_AXIAL_0.25W, symbol Device:R
- removed R410: 1.2k, MATRIX_1.4:RESISTOR_AXIAL_0.25W, symbol Device:R
- removed R411, R412: 390, MATRIX_1.4:RESISTOR_AXIAL_0.25W, symbol Device:R
- removed R413: 2.2k, MATRIX_1.4:RESISTOR_AXIAL_0.25W, symbol Device:R
- removed R4151: 120, MATRIX_1.4:RESISTOR_AXIAL_0.5W, symbol Device:R
- removed R416, R417: 5.6, MATRIX_1.4:RESISTOR_BLOCK_5W, symbol Device:R
- removed R4181, R4182, R4183, R4184, R4185, R4186, R4191, R4192, R4193, R4194, R4195, R4196: 0.33, MATRIX_1.4:RESISTOR_BLOCK_5W, symbol Device:R
- removed R420: 10, MATRIX_1.4:RESISTOR_BLOCK_5W, symbol Device:R
- removed R601, R701: 12k, MATRIX_1.4:RESISTOR_AXIAL_0.25W, symbol Device:R
- removed R602, R603, R702, R703: 120k, MATRIX_1.4:RESISTOR_AXIAL_0.25W, symbol Device:R
- removed R604, R704: 1.5k, MATRIX_1.4:RESISTOR_AXIAL_0.25W, symbol Device:R
- removed R605, R705: 56, MATRIX_1.4:RESISTOR_AXIAL_0.5W, symbol Device:R
- removed R606, R706: 1, MATRIX_1.4:RESISTOR_BLOCK_5W, symbol Device:R
- removed R608, R609, R610, R611, R612, R614, R615, R708, R709, R710, R711, R712, R714, R715: 2.7k, MATRIX_1.4:RESISTOR_AXIAL_0.25W, symbol Device:R
- removed R613, R713: 15k, MATRIX_1.4:RESISTOR_AXIAL_0.25W, symbol Device:R
- removed R616, R716: 4.7, MATRIX_1.4:RESISTOR_AXIAL_0.5W, symbol Device:R
- removed R617, R717: 27k, MATRIX_1.4:RESISTOR_AXIAL_0.25W, symbol Device:R
- removed R618, R718: 100k, MATRIX_1.4:RESISTOR_AXIAL_0.25W, symbol Device:R
- removed R619, R719: 680, MATRIX_1.4:RESISTOR_AXIAL_0.5W, symbol Device:R
- removed RT401: 5k, MATRIX_1.4:RESISTOR_ROUND_TRIMPOT_STD, symbol Device:R_Trim
- removed XQ6011, XQ6012: IRF9640, MATRIX_1.4:TO-220-MIRRORED, symbol MATRIX_1.4:Q_PMOS_DGS
- removed XQ7011, XQ7012: IRF640, MATRIX_1.4:TO-220-MIRRORED, symbol MATRIX_1.4:Q_NMOS_DGS
- added R901: 4, symbol Device:R
- added V11, V12: DC 120V, symbol pspice:VSOURCE
- added V20: dc 0 ac 1.41 sin(0 1.41 1k 0 0), symbol pspice:VSOURCE
Connections:
- net +120V: now also V11.1 (E1)
- net -120V: now also V12.2 (E2)
- net 0: now also R901.2, V11.2 (E2), V12.1 (E1), V20.2 (E2)
- net MAIN_IN: now also V20.1 (E1)
- net VPOUT: now also R901.1
Other:
- added sheet POWER-AMP (MATRIX-1.4-IV-T13-TD-DEV-3-POWER-AMP-BLOCK.kicad_sch)
- added sheet PROTECTION-SYSTEM (MATRIX-1.4-IV-PROTECTION-SYSTEM-BLOCK.kicad_sch)
- note added: "*SPICE Netlist Title .title MATRIX 1.4 IV T13 1400W RMS TD-CLASS - DEVELOPMENT RELEASE 3 * Transient analysis directive for 1KHz with input at 1.41Vp * To apply the directive, please uncomment the line below. *.tran 0.1u 1m * Fourier analysis to check the percentage of THD (Total Harmonic Distortion) * To apply the directive, please uncomment the line below. *.fourier 1k v(vmout) * AC analysis di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"
- company: MATRIX 1.4 IV T13 -> (none)
- title: 1400 WATTS RMS CLASS-TD\nAUDIO POWER AMPLIFIER\nFOR 4-OHMS LOUDSPEAKER -> (none)
